Commit message: Refactor links into reusable xacro macros

File: urdf/base/base.xacro (robot description, xacro)
@@ -1,31 +1,36 @@
 <?xml version="1.0"?>
 <robot xmlns:xacro="http://www.ros.org/wiki/xacro">
-<!-- declaring variables -->
-<xacro:property name="box_length" value="0.2"/>
-<xacro:property name="box_width" value="0.2"/>
-<xacro:property name="box_height" value="0.05"/>
-<xacro:property name="ground_offset" value="0.025"/>
+    <!-- declaring variables -->
+    <xacro:property name="box_length" value="0.2"/>
+    <xacro:property name="box_width" value="0.2"/>
+    <xacro:property name="box_height" value="0.05"/>
+    <xacro:property name="ground_offset" value="0.025"/>
+    <!-- base_footprint -->
     <link name="base_footprint"/>
-<!-- baselink defined (base_chassis) -->
-    <link name="base_link">
-        <visual>
-            <origin xyz="0 0 0" rpy="0 0 0"/>
-            <geometry>
-                <box size ="${box_length} ${box_width} ${box_height}"/>
-            </geometry>
-            <material name="green"/>
-        </visual>
-        <collision>
-            <origin xyz="0 0 0" rpy="0 0 0"/>
-            <geometry>
-                <box size="${box_length} ${box_width} ${box_height}"/>
-            </geometry>
-        </collision>
-    </link>
-<!-- joints -->
-    <joint name="base_footprint_to_base_link" type="fixed">
-        <parent link="base_footprint"/>
-        <child link="base_link"/>
-        <origin xyz="0 0 ${ground_offset + box_height/2}" rpy="0 0 0"/>
-    </joint>
+    <!-- create_box function declaration -->
+    <xacro:macro name="create_box" params="prefix length width height color">
+        <link name="${prefix}_box">
+            <visual>
+                <origin xyz="0 0 0" rpy="0 0 0"/>
+                <geometry>
+                    <box size="${length} ${width} ${height}"/>
+                </geometry>
+                <material name="${color}"/>
+            </visual>
+            <collision>
+                <origin xyz="0 0 0" rpy="0 0 0"/>
+                <geometry>
+                    <box size="${length} ${width} ${height}"/>
+                </geometry>
+            </collision>
+        </link>
+    </xacro:macro>
+        <!-- create_joint function declaration -->
+   <xacro:macro name="create_joint" params="parent_link child_link type reflect x y z roll pitch yaw">
+        <joint name="${parent_link}_to_${child_link}" type="${type}">
+            <parent link="${parent_link}"/>
+            <child link="${child_link}"/>
+            <origin xyz="${reflect * x} ${reflect * y} ${reflect * z}" rpy="${roll} ${pitch} ${yaw}"/>
+        </joint>
+    </xacro:macro>
 </robot>

File: urdf/my_bot.urdf.xacro (robot description, xacro)
@@ -1,13 +1,122 @@
 <?xml version="1.0"?>
 <robot name="my_bot" xmlns:xacro="http://www.ros.org/wiki/xacro">
-<!-- materials included -->
-<xacro:include filename="materials.xacro"/>
-<!-- base_link and base_foot_print included -->
-<xacro:include filename="base/base.xacro"/>
-<!-- drive wheels included -->
-<xacro:include filename="wheels/wheels.xacro"/>
-<!-- castor_wheels included -->
-<xacro:include filename="wheels/castor_wheels.xacro"/>
-<!-- lidar_mount and lidar included -->
-<xacro:include filename="sensors/lidar.xacro"/>
+    <!-- materials included -->
+    <xacro:include filename="materials.xacro"/>
+    <!-- base_link and base_foot_print included -->
+    <xacro:include filename="base/base.xacro"/>
+    <!-- function call to create base -->
+    <xacro:create_box
+        prefix="base_link"
+        length="${box_length}"
+        width="${box_width}"
+        height="${box_height}"
+        color="green"
+    />
+    <!-- A function call to create joint -->
+    <xacro:create_joint
+        parent_link="base_footprint"
+        child_link="base_link_box"
+        type="fixed"
+        reflect="1"
+        x ="0" y="0" z="${ground_offset + box_height/2}"
+        roll="0" pitch="0" yaw="0"
+    />
+    <!-- drive wheels included -->
+    <xacro:include filename="wheels/wheels.xacro"/>
+    <!-- A function call to create left_wheel -->
+    <xacro:create_wheel
+        prefix="left"
+        radius="${wheel_radius}"
+        width="${wheel_width}"
+        color="black"
+    />
+    <xacro:create_wheel_joint
+        parent_link="base_link_box"
+        child_link="left_wheel_link"
+        type="continuous"
+        reflect="1"
+        x ="0" y ="${box_width/2 + wheel_width/2}" z="0"
+        roll="0" pitch="0" yaw="0"
+        axis="0 1 0"
+    />
+    <!-- A function call to create left_wheel -->
+    <xacro:create_wheel
+        prefix="right"
+        radius="${wheel_radius}"
+        width="${wheel_width}"
+        color="black"
+    />
+    <xacro:create_wheel_joint
+        parent_link="base_link_box"
+        child_link="right_wheel_link"
+        type="continuous"
+        reflect="-1"
+        x ="0" y ="${box_width/2 + wheel_width/2}" z="0"
+        roll="0" pitch="0" yaw="0"
+        axis="0 1 0"
+    />
+    <!-- castor_wheels included -->
+    <xacro:include filename="wheels/castor_wheels.xacro"/>
+    <!-- A function call to create  front castor_wheel -->
+    <xacro:create_castor_wheel
+        prefix="front"
+        radius="${castor_radius}"
+        color = "black"
+    />
+    <xacro:create_wheel_joint
+        parent_link="base_link_box"
+        child_link="front_castor_wheel"
+        type="fixed"
+        reflect="1"
+        x="${castor_x_offset}" y="0" z="${-1*(box_height-castor_radius)}"
+        roll="0" pitch="0" yaw="0"
+        axis="1 1 1"
+    />
+    <!-- A function call to create rear castor_wheel -->
+    <xacro:create_castor_wheel
+        prefix="rear"
+        radius="${castor_radius}"
+        color = "black"
+    />
+    <xacro:create_wheel_joint
+        parent_link="base_link_box"
+        child_link="rear_castor_wheel"
+        type="fixed"
+        reflect="-1"
+        x="${castor_x_offset}" y="0" z="${(box_height-castor_radius)}"
+        roll="0" pitch="0" yaw="0"
+        axis="1 1 1"
+    />
+    <!-- lidar_mount and lidar included -->
+    <xacro:include filename="sensors/lidar.xacro"/>
+    <!-- A function call to create lidar_mount -->
+    <xacro:create_box
+        prefix="lidar_mount"
+        length="${lidar_mount_length}"
+        width="${lidar_mount_width}"
+        height="${lidar_mount_height}"
+        color="red"
+    />
+    <xacro:create_joint
+        parent_link="base_link_box"
+        child_link="lidar_mount_box"
+        type="fixed"
+        reflect="1"
+        x="${lidar_mount_x_offset}" y="0" z="${box_height/2 + lidar_mount_height/2}"
+        roll="0" pitch="0" yaw="0"
+    />
+<!-- A function call to spawn lidar -->
+    <xacro:spawn_lidar
+        radius="${lidar_radius}"
+        height="${lidar_height}"
+        color="blue"
+    />
+    <xacro:create_joint
+        parent_link="lidar_mount_box"
+        child_link="lidar"
+        type="fixed"
+        reflect="1"
+        x="0" y="0" z="${lidar_mount_height/2 + lidar_height/2}"
+        roll="0" pitch="0" yaw="0"
+    />
 </robot>

File: urdf/sensors/lidar.xacro (robot description, xacro)
@@ -1,51 +1,27 @@
 <?xml version="1.0"?>
 <robot xmlns:xacro="http://www.ros.org/wiki/xacro">
-<!-- lidar and lidar_mount properties -->
-<xacro:property name="lidar_mount_length" value="0.07"/>
-<xacro:property name="lidar_mount_width" value="0.06"/>
-<xacro:property name="lidar_mount_height" value="0.045"/>
-<xacro:property name="lidar_mount_x_offset" value="0.035"/>
-<xacro:property name="lidar_radius" value="0.0295"/>
-<xacro:property name="lidar_height" value="0.02"/>
-    <!-- lidar_mount_definition -->
-<link name="lidar_mount">
-    <visual>
-    <origin xyz="0 0 0" rpy="0 0 0"/>
-        <geometry>
-            <box size="${lidar_mount_length} ${lidar_mount_width} ${lidar_mount_height}"/>
-        </geometry>
-        <material name="black"/>
-    </visual>
-    <collision>
-    <origin xyz="0 0 0" rpy="0 0 0"/>
-        <geometry>
-            <box size="${lidar_mount_length} ${lidar_mount_width} ${lidar_mount_height}"/>
-        </geometry>
-    </collision>
-</link>
-<joint name="base_link_to_lidar_mount" type="fixed">
-    <parent link="base_link"/>
-    <child link="lidar_mount"/>
-    <origin xyz="${lidar_mount_x_offset} 0.0 ${box_height/2 + lidar_mount_height/2}"/>
-</joint>
-<link name="lidar">
-    <visual>
-        <origin xyz="0 0 0"/>
-        <geometry>
-            <cylinder radius="${lidar_radius}" length="${lidar_height}"/>
-        </geometry>
-        <material name="blue"/>
-    </visual>
-    <collision>
-        <origin xyz="0 0 0"/>
-        <geometry>
-            <cylinder radius="${lidar_radius}" length="${lidar_height}"/>
-        </geometry>
-    </collision>
-</link>
-<joint name="lidar_mount_to_mount" type="fixed">
-    <parent link="lidar_mount"/>
-    <child link="lidar"/>
-    <origin xyz="0 0 ${lidar_mount_height/2 + lidar_height/2}" rpy="0 0 0"/>
-</joint>
+    <!-- lidar and lidar_mount properties -->
+    <xacro:property name="lidar_mount_length" value="0.07"/>
+    <xacro:property name="lidar_mount_width" value="0.06"/>
+    <xacro:property name="lidar_mount_height" value="0.045"/>
+    <xacro:property name="lidar_mount_x_offset" value="0.035"/>
+    <xacro:property name="lidar_radius" value="0.0295"/>
+    <xacro:property name="lidar_height" value="0.02"/>
+    <xacro:macro name="spawn_lidar" params="radius height color">
+        <link name="lidar">
+            <visual>
+                <origin xyz="0.0 0.0 0.0" rpy="0.0 0.0 0.0"/>
+            <geometry>
+                <cylinder radius="${radius}" length="${height}"/>
+            </geometry>
+            <material name="${color}"/>
+            </visual>
+            <collision>
+                <origin xyz="0.0 0.0 0.0" rpy="0.0 0.0 0.0"/>
+                <geometry>
+                    <cylinder radius="${radius}" length="${height}"/>
+                </geometry>
+            </collision>
+        </link>
+    </xacro:macro>
 </robot>

File: urdf/wheels/castor_wheels.xacro (robot description, xacro)
@@ -4,44 +4,21 @@
 <xacro:property name="castor_radius" value="0.012"/>
 <xacro:property name="castor_x_offset" value="0.075"/>
-<!-- castor wheels definiton -->
-    <link name="front_castor_wheel">
-    <visual>
-        <origin xyz="0 0 0" rpy="0 0 0"/>
-        <geometry>
-            <sphere radius="${castor_radius}"/>
-        </geometry>
-        <material name="blue"/>
-    </visual>
-    <collision>
-        <origin xyz="0 0 0" rpy="0 0 0"/>
-        <geometry>
-            <sphere radius="${castor_radius}"/>
-        </geometry>
-    </collision>
-    </link>
-    <joint name="base_link_to_front_castor_wheel" type="fixed">
-        <parent link="base_link"/>
-        <child link="front_castor_wheel"/>
-        <origin xyz ="${castor_x_offset} 0 ${-1*(box_height-castor_radius)}" rpy="0 0 0"/>
-    </joint>
-    <link name="rear_castor_wheel">
-    <visual>
-        <origin xyz="0 0 0" rpy="0 0 0"/>
-        <geometry>
-            <sphere radius="${castor_radius}"/>
-        </geometry>
-        <material name="black"/>
-    </visual>
-    <collision>
-        <origin xyz="0 0 0" rpy="0 0 0"/>
-        <geometry>
-            <sphere radius="${castor_radius}"/>
-        </geometry>
-    </collision>
-    </link>
-    <joint name="base_link_to_rear_castor_wheel" type="fixed">
-        <parent link="base_link"/>
-        <child link="rear_castor_wheel"/>
-        <origin xyz ="${-1*(castor_x_offset)} 0 ${-1*(ground_offset + box_height/2 - castor_radius)}" rpy="0 0 0"/>
-    </joint>
+<!-- A function declaration for a castor_wheel -->
+    <xacro:macro name="create_castor_wheel" params="prefix radius color">
+        <link name="${prefix}_castor_wheel">
+            <visual>
+                <origin xyz="0.0 0.0 0.0" rpy="0.0 0.0 0.0"/>
+                <geometry>
+                    <sphere radius="${radius}"/>
+                </geometry>
+                <material name="${color}"/>
+            </visual>
+            <collision>
+                <origin xyz="0.0 0.0 0.0" rpy="0.0 0.0 0.0"/>
+                <geometry>
+                    <sphere radius="${radius}"/>
+                </geometry>
+            </collision>
+        </link>
+    </xacro:macro>
 </robot>

File: urdf/wheels/wheels.xacro (robot description, xacro)
@@ -1,50 +1,32 @@
 <?xml version="1.0"?>
 <robot xmlns:xacro="http://www.ros.org/wiki/xacro">
-<!-- Properties declaarations -->
-<xacro:property name="wheel_radius" value="0.05"/>
-<xacro:property name="wheel_width" value="0.025"/>
-        <!-- left_wheel link defined -->
-    <link name="left_wheel_link">
-    <visual>
-        <origin xyz="0 0 0" rpy="${pi/2} 0 0"/>
-        <geometry>
-            <cylinder radius="${wheel_radius}" length="${wheel_width}"/>
-        </geometry>
-        <material name="black"/>
-    </visual>
-    <collision>
-        <origin xyz="0 0 0" rpy="${pi/2} 0 0"/>
-        <geometry>
-            <cylinder radius="${wheel_radius}" length="${wheel_width}"/>
-        </geometry>
-    </collision>
-    </link>
-    <joint name="base_link_to_left_wheel" type="continuous">
-        <parent link="base_link"/>
-        <child link="left_wheel_link"/>
-        <origin xyz="0 ${box_width/2 + wheel_width/2} 0" rpy="0 0 0"/>
-        <axis xyz="0.0 1.0 0.0"/>
-    </joint>
-    <!-- right_wheel link defined -->
-    <link name="right_wheel_link">
-        <visual>
-            <origin xyz="0 0 0" rpy="${pi/2} 0 0"/>
-            <geometry>
-                <cylinder radius="${wheel_radius}" length="${wheel_width}"/>
-            </geometry>
-            <material name="red"/>
-        </visual>
-        <collision>
-            <origin xyz="0 0 0" rpy="${pi/2} 0 0"/>
-            <geometry>
-                <cylinder radius="${wheel_radius}" length="${wheel_width}"/>
-            </geometry>
-        </collision>
-    </link>
-    <joint name="base_link_to_right_wheel" type="continuous">
-        <parent link="base_link"/>
-        <child link="right_wheel_link"/>
-        <origin xyz="0 ${-1*(box_length/2 + wheel_width/2)} 0" rpy="0 0 0"/>
-        <axis xyz="0.0 1.0 0.0"/>
-    </joint>
+    <!-- Properties declaarations -->
+    <xacro:property name="wheel_radius" value="0.05"/>
+    <xacro:property name="wheel_width" value="0.025"/>
+    <xacro:macro name="create_wheel" params="prefix radius width color">
+        <link name="${prefix}_wheel_link">
+            <visual>
+                <origin xyz="0 0 0" rpy="${pi/2} 0 0"/>
+                <geometry>
+                    <cylinder radius="${radius}" length="${width}"/>
+                </geometry>
+                <material name="${color}"/>
+            </visual>
+            <collision>
+                <origin xyz="0 0 0" rpy="${pi/2} 0 0"/>
+                <geometry>
+                    <cylinder radius="${radius}" length="${width}"/>
+                </geometry>
+            </collision>
+        </link>
+    </xacro:macro>
+    <!-- create_wheel_joint function declaration -->
+   <xacro:macro name="create_wheel_joint" params="parent_link child_link type reflect x y z roll pitch yaw axis">
+        <joint name="${parent_link}_to_${child_link}" type="${type}">
+            <parent link="${parent_link}"/>
+            <child link="${child_link}"/>
+            <origin xyz="${reflect * x} ${reflect * y} ${reflect * z}" rpy="${roll} ${pitch} ${yaw}"/>
+            <axis xyz="${axis}"/>
+        </joint>
+    </xacro:macro>
 </robot>
