Commit message: included cargo and extended lidar_mount

File: urdf/my_bot.urdf.xacro (robot description, xacro)
@@ -120,3 +120,19 @@
         roll="0" pitch="0" yaw="0"
     />
+    <xacro:include filename="cargo/cargo.xacro"/>
+    <xacro:create_box
+        prefix="cargo"
+        length="${cargo_length}"
+        width="${cargo_width}"
+        height="${cargo_height}"
+        color="black"
+    />
+    <xacro:create_joint
+        parent_link="base_link_box"
+        child_link="cargo_box"
+        type="fixed"
+        reflect="1"
+        x="${-lidar_mount_width/2}" y="0" z="${box_height/2 + cargo_height/2}"
+        roll="0" pitch="0" yaw="0"
+    />
 </robot>

File: urdf/sensors/lidar.xacro (robot description, xacro)
@@ -2,8 +2,8 @@
 <robot xmlns:xacro="http://www.ros.org/wiki/xacro">
     <!-- lidar and lidar_mount properties -->
-    <xacro:property name="lidar_mount_length" value="0.07"/>
-    <xacro:property name="lidar_mount_width" value="0.06"/>
-    <xacro:property name="lidar_mount_height" value="0.045"/>
-    <xacro:property name="lidar_mount_x_offset" value="0.035"/>
+    <xacro:property name="lidar_mount_length" value="0.035"/>
+    <xacro:property name="lidar_mount_width" value="0.035"/>
+    <xacro:property name="lidar_mount_height" value="0.150"/>
+    <xacro:property name="lidar_mount_x_offset" value="0.0825"/>
     <xacro:property name="lidar_radius" value="0.0295"/>
     <xacro:property name="lidar_height" value="0.02"/>
